File: ddr.sch (KiCad schematic (older format))
At the start: 1 part

Commit message: ddr is confusing
Parts:
- added J?: 2-2013310-2, 220133102, symbol 2-2013310-2:2-2013310-2
Connections:
- net RAS#: now reaches U?.A10 (DDR_RASN)
- net RAS#: now also J?.157
- net A0: now reaches U?.A11 (DDR_A0)
- net A0: now also J?.151
- net CK0#: now reaches U?.A13 (DDR_CLKN)
- net CK0#: now also J?.52
- net A5: now reaches U?.A14 (DDR_A5)
- net A5: now also J?.46
- net A15: now reaches U?.A16 (DDR_A15)
- net A15: now also J?.141
- net DQ18: now reaches U?.A17 (DDR_DQ18)
- net DQ18: now also J?.26
- net DQS2#: now reaches U?.A19 (DDR_DQS2N)
- net DQS2#: now also J?.23
- net DM0: now reaches U?.A2 (DDR_DM3)
- net DM0: now also J?.6
- net DQ19: now reaches U?.A20 (DDR_DQ19)
- net DQ19: now also J?.27
- net DQS0#: now reaches U?.A22 (DDR_DQS0N)
- net DQS0#: now also J?.107
- net DQ4: now reaches U?.A23 (DDR_DQ4)
- net DQ4: now also J?.104
- net DQS3#: now reaches U?.A4 (DDR_DQS3N)
- net DQS3#: now also J?.133
- net DQ31: now reaches U?.A5 (DDR_DQ31)
- net DQ31: now also J?.137
- net DQS1#: now reaches U?.A7 (DDR_DQS1N)
- net DQS1#: now also J?.14
- net CK1: now reaches U?.A8 (DDR_CS0N)
- net CK1: now also J?.153
- net CAS#: now reaches U?.B10 (DDR_CASN)
- net CAS#: now also J?.58
- net BA0: now reaches U?.B11 (DDR_BA2)
- net BA0: now also J?.55
- net A2: now reaches U?.B12 (DDR_A2)
- net A2: now also J?.150
- net CK0: now reaches U?.B13 (DDR_CLK)
- net CK0: now also J?.51
- net A6: now reaches U?.B14 (DDR_A6)
- net A6: now also J?.147
- net A11: now reaches U?.B15 (DDR_A11)
- net A11: now also J?.144
- net A14: now reaches U?.B16 (DDR_A14)
- net A14: now also J?.142
- net DQ17: now reaches U?.B17 (DDR_DQ17)
- net DQ17: now also J?.21
- net DQ21: now reaches U?.B18 (DDR_DQ21)
- net DQ21: now also J?.123
- net DQS2: now reaches U?.B19 (DDR_DQS2)
- net DQS2: now also J?.24
- net DQ24: now reaches U?.B2 (DDR_DQ24)
- net DQ24: now also J?.29
- net DQ22: now reaches U?.B20 (DDR_DQ22)
- net DQ22: now also J?.127
- net DQ23: now reaches U?.B21 (DDR_DQ23)
- net DQ23: now also J?.128
- net DQS0: now reaches U?.B22 (DDR_DQS0)
- net DQS0: now also J?.108
- net DQ5: now reaches U?.B23 (DDR_DQ5)
- net DQ5: now also J?.105
- net DQ25: now reaches U?.B3 (DDR_DQ25)
- net DQ25: now also J?.30
- net DQS3: now reaches U?.B4 (DDR_DQS3)
- net DQS3: now also J?.134
- net DQ30: now reaches U?.B5 (DDR_DQ30)
- net DQ30: now also J?.136
- net DQ10: now reaches U?.B6 (DDR_DQ10)
- net DQ10: now also J?.17
- net DQS1: now reaches U?.B7 (DDR_DQS1)
- net DQS1: now also J?.15
- net CKE1: now reaches U?.B8 (DDR_CKE1)
- net CKE1: now also J?.139
- net CK1#: now reaches U?.B9 (DDR_CS1N)
- net CK1#: now also J?.154
- net WE#: now reaches U?.C10 (DDR_WEN)
- net WE#: now also J?.57
- net BA1: now reaches U?.C11 (DDR_BA1)
- net BA1: now also J?.156
- net A1: now reaches U?.C12 (DDR_A1)
- net A1: now also J?.49
- net A4: now reaches U?.C13 (DDR_A4)
- net A4: now also J?.148
- net A7: now reaches U?.C14 (DDR_A7)
- net A7: now also J?.145
- net A10: now reaches U?.C15 (DDR_A10)
- net A10: now also J?.54
- net A13: now reaches U?.C16 (DDR_A13)
- net A13: now also J?.60
- net ODT1: now reaches U?.C17 (DDR_ODT1)
- net DQ16: now reaches U?.C18 (DDR_DQ16)
- net DQ16: now also J?.20
- net DQ20: now reaches U?.C19 (DDR_DQ20)
- net DQ20: now also J?.122
- net DM1: now reaches U?.C20 (DDR_DM2)
- net DM1: now also J?.116
- net DQ2: now reaches U?.C22 (DDR_DQ2)
- net DQ2: now also J?.8
- net DQ26: now reaches U?.C3 (DDR_DQ26)
- net DQ26: now also J?.34
- net DQ27: now reaches U?.C4 (DDR_DQ27)
- net DQ27: now also J?.35
- net DQ29: now reaches U?.C5 (DDR_DQ29)
- net DQ29: now also J?.131
- net DQ9: now reaches U?.C6 (DDR_DQ9)
- net DQ9: now also J?.12
- net DQ12: now reaches U?.C7 (DDR_DQ12)
- net DQ12: now also J?.113
- net DQ15: now reaches U?.C8 (DDR_DQ15)
- net DQ15: now also J?.120
- net CKE0: now reaches U?.C9 (DDR_CKE0)
- net CKE0: now also J?.37
- net BA2: now reaches U?.D11 (DDR_BA0)
- net BA2: now also J?.40
- net A8: now reaches U?.D14 (DDR_A8)
- net A8: now also J?.45
- net ODT0: now reaches U?.D17 (DDR_ODT0)
- net ODT0: now also J?.160
- net A12: now reaches U?.D18 (DDR_A12)
- net A12: now also J?.42
- net DM3: now reaches U?.D20 (DDR_DM0)
- net DM3: now also J?.32
- net DQ1: now reaches U?.D21 (DDR_DQ1)
- net DQ1: now also J?.4
- net DQ3: now reaches U?.D22 (DDR_DQ3)
- net DQ3: now also J?.9
- net DQ6: now reaches U?.D23 (DDR_DQ6)
- net DQ6: now also J?.110
- net DQ28: now reaches U?.D5 (DDR_DQ28)
- net DQ28: now also J?.130
- net DQ8: now reaches U?.D6 (DDR_DQ8)
- net DQ8: now also J?.11
- net DQ14: now reaches U?.D8 (DDR_DQ14)
- net DQ14: now also J?.119
- net RESET#: now reaches U?.E11 (DDR_RESETN)
- net RESET#: now also J?.117
- net A3: now reaches U?.E13 (DDR_A3)
- net A3: now also J?.48
- net A9: now reaches U?.E14 (DDR_A9)
- net A9: now also J?.43
- net DQ0: now reaches U?.E22 (DDR_DQ0)
- net DQ0: now also J?.3
- net DQ7: now reaches U?.E23 (DDR_DQ7)
- net DQ7: now also J?.111
- net DM2: now reaches U?.E6 (DDR_DM1)
- net DM2: now also J?.125
- net DQ11: now reaches U?.E7 (DDR_DQ11)
- net DQ11: now also J?.18
- net DQ13: now reaches U?.E8 (DDR_DQ13)
- net DQ13: now also J?.114
- new net DM4: J?.170
- new net DM5: J?.77
- new net DM6: J?.187
- new net DM7: J?.94
- new net DQ32: J?.65
- new net DQ33: J?.66
- new net DQ34: J?.71
- new net DQ35: J?.72
- new net DQ36: J?.167
- new net DQ37: J?.168
- new net DQ38: J?.172
- new net DQ39: J?.173
- new net DQ40: J?.74
- new net DQ41: J?.75
- new net DQ42: J?.79
- new net DQ43: J?.80
- new net DQ44: J?.175
- new net DQ45: J?.176
- new net DQ46: J?.181
- new net DQ47: J?.182
- new net DQ48: J?.82
- new net DQ49: J?.83
- new net DQ50: J?.88
- new net DQ51: J?.89
- new net DQ52: J?.184
- new net DQ53: J?.185
- new net DQ54: J?.189
- new net DQ55: J?.190
- new net DQ56: J?.91
- new net DQ57: J?.92
- new net DQ58: J?.96
- new net DQ59: J?.97
- new net DQ60: J?.192
- new net DQ61: J?.193
- new net DQ62: J?.198
- new net DQ63: J?.199
- new net DQS4: J?.69
- new net DQS4#: J?.68
- new net DQS5: J?.179
- new net DQS5#: J?.178
- new net DQS6: J?.86
- new net DQS6#: J?.85
- new net DQS7: J?.196
- new net DQS7#: J?.195
- new net NC: J?.162, J?.163, J?.39, J?.61, J?.63
- new net NF: J?.201
- new net S0#: J?.159
- new net SA0: J?.99
- new net SA1: J?.101
- new net SCL: J?.203
- new net SDA: J?.202
- new net VDD: J?.140, J?.143, J?.146, J?.149, J?.152, J?.155, J?.158, J?.161, J?.164, J?.38, J?.41, J?.44, J?.47, J?.50, J?.53, J?.56, J?.59, J?.62
- new net VDDSPD: J?.100
- new net VREFCA: J?.165
- new net VREFDQ: J?.1
- new net VSS: J?.10, J?.103, J?.106, J?.109, J?.112, J?.115, J?.118, J?.121, J?.124, J?.126, J?.129, J?.13, J?.132, J?.135, J?.138, J?.16, J?.166, J?.169, J?.171, J?.174, J?.177, J?.180, J?.183, J?.186, J?.188, J?.19, J?.191, J?.194, J?.197, J?.2, J?.200, J?.22, J?.25, J?.28, J?.31, J?.33, J?.36, J?.5, J?.64, J?.67, J?.7, J?.70, J?.73, J?.76, J?.78, J?.81, J?.84, J?.87, J?.90, J?.93, J?.95, J?.98
- new net VTT: J?.102, J?.204
Other:
- moved on the sheet: U?C
